File: ergogen/output/pcbs/oregano.kicad_pcb (KiCad board)
At the start: 2 copper layers, 150.3 x 106.6 mm, 52 parts

Commit message: Many men
Connections:
- DISP1 pad 10: CS -> P1
- DISP1 pad 20: CS -> P1

Commit message: Add routed pcb; Remove zip
Connections:
- net sw1 renamed BAT_P
Other:
- outline, holes or cut-outs redrawn
Changed lines of the file:
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@@
   (title_block
     (title "oregano")
-    (date "2026-04-01")
+    (date "2026-04-02")
     (rev "v1.0.0")
     (company "Unknown")
@@
 (net 74 "DISP1_4")
 (net 75 "DISP1_5")
-(net 76 "sw1")
+(net 76 "BAT_P")
 (net 77 "JST1_1")
 (net 78 "JST1_2")
@@
             (net 78 "JST1_2")
         )
-        (pad "1" smd custom (at -1 2.816 450) (size 1.2 0.5) (layers "F.Cu" "F.Mask" "F.Paste") (net 76 "sw1")
+        (pad "1" smd custom (at -1 2.816 450) (size 1.2 0.5) (layers "F.Cu" "F.Mask" "F.Paste") (net 76 "BAT_P")
             (clearance 0.1) (zone_connect 0)
             (options (clearance outline) (anchor rect))
@@
             )
         )
-        (pad "1" smd custom (at 1 2.816 450) (size 1.2 0.5) (layers "B.Cu" "B.Mask" "B.Paste") (net 76 "sw1")
+        (pad "1" smd custom (at 1 2.816 450) (size 1.2 0.5) (layers "B.Cu" "B.Mask" "B.Paste") (net 76 "BAT_P")
             (clearance 0.1) (zone_connect 0)
             (options (clearance outline) (anchor rect))
@@
             (pad "" np_thru_hole circle (at -1.5 0.33 115.4) (size 0.9 0.9) (drill 0.9) (layers *.Cu *.Mask))
             (pad "" np_thru_hole circle (at 1.5 0.33 115.4) (size 0.9 0.9) (drill 0.9) (layers *.Cu *.Mask))
-            (pad 1 smd rect (at -2.25 -1.43 115.4) (size 0.7 1.5) (layers F.Cu F.Paste F.Mask) (net 76 "sw1"))
+            (pad 1 smd rect (at -2.25 -1.43 115.4) (size 0.7 1.5) (layers F.Cu F.Paste F.Mask) (net 76 "BAT_P"))
             (pad 2 smd rect (at 0.75 -1.43 115.4) (size 0.7 1.5) (layers F.Cu F.Paste F.Mask) (net 34 "RAW"))
             (pad "" smd rect (at 2.25 -1.43 115.4) (size 0.7 1.5) (layers F.Cu F.Paste F.Mask))
@@
             (pad "" np_thru_hole circle (at -1.5 0.33 115.4) (size 0.9 0.9) (drill 0.9) (layers *.Cu *.Mask))
             (pad "" np_thru_hole circle (at 1.5 0.33 115.4) (size 0.9 0.9) (drill 0.9) (layers *.Cu *.Mask))
-            (pad 1 smd rect (at 2.25 -1.43 115.4) (size 0.7 1.5) (layers B.Cu B.Paste B.Mask) (net 76 "sw1"))
+            (pad 1 smd rect (at 2.25 -1.43 115.4) (size 0.7 1.5) (layers B.Cu B.Paste B.Mask) (net 76 "BAT_P"))
             (pad 2 smd rect (at -0.75 -1.43 115.4) (size 0.7 1.5) (layers B.Cu B.Paste B.Mask) (net 34 "RAW"))
             (pad "" smd rect (at -2.25 -1.43 115.4) (size 0.7 1.5) (layers B.Cu B.Paste B.Mask))
@@
     (fp_circle (center 0 0) (end -2.1500000000000004 0) (layer "B.CrtYd") (stroke (width 0.05) (type solid)) (fill none))
   )
-  (gr_line (start 59.411155977272735 104) (end 120.13990954870408 104) (layer Edge.Cuts) (stroke (width 0.15) (type default)))
-(gr_line (start 57.41321888201499 102.09081540432976) (end 57.086781117985 94.90918459567001) (layer Edge.Cuts) (stroke (width 0.15) (type default)))
-(gr_line (start 55.08884402272727 93) (end 41 93) (layer Edge.Cuts) (stroke (width 0.15) (type default)))
+  (gr_line (start 59.5 104) (end 120.13990954870408 104) (layer Edge.Cuts) (stroke (width 0.15) (type default)))
+(gr_line (start 57.5 102) (end 57.5 95) (layer Edge.Cuts) (stroke (width 0.15) (type default)))
+(gr_line (start 55.5 93) (end 41 93) (layer Edge.Cuts) (stroke (width 0.15) (type default)))
 (gr_line (start 39 91) (end 39 56.5) (layer Edge.Cuts) (stroke (width 0.15) (type default)))
-(gr_line (start 41 54.5) (end 55.14793769230769 54.5) (layer Edge.Cuts) (stroke (width 0.15) (type default)))
-(gr_line (start 57.14204669230769 52.65339300000005) (end 57.3579533076923 49.84660700000006) (layer Edge.Cuts) (stroke (width 0.15) (type default)))
-(gr_line (start 59.352062307692314 48) (end 73.57544438461538 48) (layer Edge.Cuts) (stroke (width 0.15) (type default)))
-(gr_line (start 75.57396668476309 46.0768661961597) (end 75.92603331523691 36.92313380384053) (layer Edge.Cuts) (stroke (width 0.15) (type default)))
-(gr_line (start 77.92455561538462 35) (end 92.19002486 35) (layer Edge.Cuts) (stroke (width 0.15) (type default)))
-(gr_line (start 94.18009926 33.199007399999914) (end 94.31990074000001 31.80099259999986) (layer Edge.Cuts) (stroke (width 0.15) (type default)))
-(gr_line (start 96.30997513999999 30) (end 114.65973424999999 30) (layer Edge.Cuts) (stroke (width 0.15) (type default)))
-(gr_line (start 116.65282575068966 31.833909008275896) (end 116.84717424931036 34.16609099172433) (layer Edge.Cuts) (stroke (width 0.15) (type default)))
-(gr_line (start 118.84026575000001 36) (end 173.5 36) (layer Edge.Cuts) (stroke (width 0.15) (type default)))
+(gr_line (start 41 54.5) (end 55.5 54.5) (layer Edge.Cuts) (stroke (width 0.15) (type default)))
+(gr_line (start 57.5 52.5) (end 57.5 50) (layer Edge.Cuts) (stroke (width 0.15) (type default)))
+(gr_line (start 59.5 48) (end 74 48) (layer Edge.Cuts) (stroke (width 0.15) (type default)))
+(gr_line (start 76 46) (end 76 37) (layer Edge.Cuts) (stroke (width 0.15) (type default)))
+(gr_line (start 78 35) (end 92.5 35) (layer Edge.Cuts) (stroke (width 0.15) (type default)))
+(gr_line (start 94.5 33) (end 94.5 32) (layer Edge.Cuts) (stroke (width 0.15) (type default)))
+(gr_line (start 96.5 30) (end 114.5 30) (layer Edge.Cuts) (stroke (width 0.15) (type default)))
+(gr_line (start 116.5 32) (end 116.5 34) (layer Edge.Cuts) (stroke (width 0.15) (type default)))
+(gr_line (start 118.5 36) (end 173.5 36) (layer Edge.Cuts) (stroke (width 0.15) (type default)))
 (gr_line (start 175.5 38) (end 175.5 91.54881869124944) (layer Edge.Cuts) (stroke (width 0.15) (type default)))
 (gr_line (start 175.69370659999998 92.40748289124934) (end 189.0811544275359 120.56943476699826) (layer Edge.Cuts) (stroke (width 0.15) (type default)))
@@
 (gr_line (start 142.20075540695547 113.85321328743969) (end 124.8919130391206 110.1543303450141) (layer Edge.Cuts) (stroke (width 0.15) (type default)))
 (gr_line (start 123.44987235979366 108.9336054973214) (end 121.99991122803107 105.26488524769272) (layer Edge.Cuts) (stroke (width 0.15) (type default)))
-(gr_arc (start 57.41321887727273 102.0908154) (mid 58.029423477272736 103.4459652) (end 59.411155977272735 104) (layer Edge.Cuts) (stroke (width 0.15) (type default)))
-(gr_arc (start 57.086781122727274 94.9091846) (mid 56.47057652272727 93.5540348) (end 55.08884402272727 93) (layer Edge.Cuts) (stroke (width 0.15) (type default)))
+(gr_arc (start 57.5 102) (mid 58.0857864 103.4142136) (end 59.5 104) (layer Edge.Cuts) (stroke (width 0.15) (type default)))
+(gr_arc (start 57.5 95) (mid 56.9142136 93.5857864) (end 55.5 93) (layer Edge.Cuts) (stroke (width 0.15) (type default)))
 (gr_arc (start 39 91) (mid 39.5857864 92.4142136) (end 41 93) (layer Edge.Cuts) (stroke (width 0.15) (type default)))
 (gr_arc (start 41 54.5) (mid 39.5857864 55.0857864) (end 39 56.5) (layer Edge.Cuts) (stroke (width 0.15) (type default)))
-(gr_arc (start 55.14793769230769 54.5) (mid 56.506836892307696 53.9674444) (end 57.142046692307694 52.653393) (layer Edge.Cuts) (stroke (width 0.15) (type default)))
-(gr_arc (start 59.352062307692314 48) (mid 57.99316310769231 48.5325556) (end 57.35795330769231 49.846607) (layer Edge.Cuts) (stroke (width 0.15) (type default)))
-(gr_arc (start 73.57544438461538 48) (mid 74.96221538461538 47.4411337) (end 75.57396678461538 46.0768662) (layer Edge.Cuts) (stroke (width 0.15) (type default)))
-(gr_arc (start 77.92455561538462 35) (mid 76.53778461538462 35.5588663) (end 75.92603321538462 36.9231338) (layer Edge.Cuts) (stroke (width 0.15) (type default)))
-(gr_arc (start 92.19002486 35) (mid 93.53203556 34.482905099999996) (end 94.18009925999999 33.1990074) (layer Edge.Cuts) (stroke (width 0.15) (type default)))
-(gr_arc (start 96.30997513999999 30) (mid 94.96796443999999 30.5170949) (end 94.31990074 31.8009926) (layer Edge.Cuts) (stroke (width 0.15) (type default)))
-(gr_arc (start 116.65282574999999 31.833909) (mid 116.01395324999999 30.5282354) (end 114.65973424999999 30) (layer Edge.Cuts) (stroke (width 0.15) (type default)))
-(gr_arc (start 116.84717425000001 34.166091) (mid 117.48604675000001 35.4717646) (end 118.84026575000001 36) (layer Edge.Cuts) (stroke (width 0.15) (type default)))
+(gr_arc (start 55.5 54.5) (mid 56.9142136 53.9142136) (end 57.5 52.5) (layer Edge.Cuts) (stroke (width 0.15) (type default)))
+(gr_arc (start 59.5 48) (mid 58.0857864 48.5857864) (end 57.5 50) (layer Edge.Cuts) (stroke (width 0.15) (type default)))
+(gr_arc (start 74 48) (mid 75.4142136 47.4142136) (end 76 46) (layer Edge.Cuts) (stroke (width 0.15) (type default)))
+(gr_arc (start 78 35) (mid 76.5857864 35.5857864) (end 76 37) (layer Edge.Cuts) (stroke (width 0.15) (type default)))
+(gr_arc (start 92.5 35) (mid 93.9142136 34.4142136) (end 94.5 33) (layer Edge.Cuts) (stroke (width 0.15) (type default)))
+(gr_arc (start 96.5 30) (mid 95.0857864 30.5857864) (end 94.5 32) (layer Edge.Cuts) (stroke (width 0.15) (type default)))
+(gr_arc (start 116.5 32) (mid 115.9142136 30.5857864) (end 114.5 30) (layer Edge.Cuts) (stroke (width 0.15) (type default)))
+(gr_arc (start 116.5 34) (mid 117.0857864 35.4142136) (end 118.5 36) (layer Edge.Cuts) (stroke (width 0.15) (type default)))
 (gr_arc (start 175.5 38) (mid 174.9142136 36.5857864) (end 173.5 36) (layer Edge.Cuts) (stroke (width 0.15) (type default)))
 (gr_arc (start 175.5 91.54881869124944) (mid 175.5490276 91.98893979124944) (end 175.6937066 92.40748289124944) (layer Edge.Cuts) (stroke (width 0.15) (type default)))
