File: routed-pcb/oregano_routed.kicad_pcb (KiCad board)
At the start: 2 copper layers, 150.3 x 106.6 mm, 52 parts

Commit message: Final routed PCB; Generate Gerbers; Ordered version
Parts:
- moved T1 0.50 mm to (176.5, 100.0)
Routing:
- net GND: track 70.3 -> 162.6 mm, vias 0 -> 2
- net P1: track 9.84 -> 71.3 mm, vias 0 -> 1
- net P3: track 9.84 -> 62.1 mm, vias 0 -> 1
- net P2: track 9.84 -> 60.9 mm, vias 0 -> 1
- net P10: track 117.1 -> 120.1 mm
- net RAW: track 80.3 -> 83.0 mm
- net BAT_P: track 34.1 -> 31.9 mm
- net VCC: track 52.4 -> 51.4 mm
- net P8: track 100.3 -> 99.3 mm
- net P15: track 172.6 -> 173.5 mm
- net P6: track 273.2 -> 272.3 mm
- net P7: track 117.6 -> 116.8 mm
- net P16: track 152.3 -> 153.0 mm
Other:
- board text added: "Linux Academic Group 2026"
- board text added: "Oregano by Pawluk"
